File: Hardware/lcd_Daughterboard.sch (KiCad schematic (older format))
At the start: 7 parts, among them J1 Conn_01x12, J2 Conn_01x12, Q1 MMBT3904, U1 ILI9341_SPI_Bare

Commit message: PCB Updated to incorporate LCD daughterboard
Parts:
- R1: value 220 -> 270
- R2: value 1k -> 1k1
- R3: value 100 -> 120
Other:
- note added: "8.61V"
- note added: "80mA from VCC to Collector"
- note added: "9.42V"
- note removed: "9.1V"
- note removed: "9.8V"
- note removed: "90mA from VCC to Collector"
Changed lines of the file:
@@
 P 6350 2500
 F 0 "R3" H 6420 2546 50  0000 L CNN
-F 1 "100" H 6420 2455 50  0000 L CNN
+F 1 "120" H 6420 2455 50  0000 L CNN
 F 2 "Resistors_SMD:R_0805_HandSoldering" V 6280 2500 50  0001 C CNN
 F 3 "~" H 6350 2500 50  0001 C CNN
@@
 P 5750 1600
 F 0 "R1" H 5820 1646 50  0000 L CNN
-F 1 "220" H 5820 1555 50  0000 L CNN
+F 1 "270" H 5820 1555 50  0000 L CNN
 F 2 "Resistors_SMD:R_0805_HandSoldering" V 5680 1600 50  0001 C CNN
 F 3 "~" H 5750 1600 50  0001 C CNN
@@
 P 5750 2500
 F 0 "R2" H 5820 2546 50  0000 L CNN
-F 1 "1k" H 5820 2455 50  0000 L CNN
+F 1 "1k1" H 5820 2455 50  0000 L CNN
 F 2 "Resistors_SMD:R_0805_HandSoldering" V 5680 2500 50  0001 C CNN
 F 3 "~" H 5750 2500 50  0001 C CNN
@@
 Connection ~ 2950 2050
 Text Notes 5800 2000 0    50   ~ 0
-9.8V
+9.42V
 Text Notes 6450 2300 0    50   ~ 0
-9.1V
+8.61V
 Text Notes 6350 1600 0    50   ~ 0
-90mA from VCC to Collector
+80mA from VCC to Collector
 $Comp
 L Connector_Generic:Conn_01x12 J1
