File: Hardware_v2/lcd_Daughterboard.kicad_sch (KiCad schematic)
At the start: 5 parts, among them J3 Conn_01x03_Pin, J4 Conn_01x03_Pin, J5 Conn_01x02_Pin, J6 Conn_01x02_Pin, U1 ILI9341_SPI_Bare

Commit message: Routing of component board
Parts:
- J4: footprint Connector_PinHeader_2.54mm:PinHeader_1x02_P2.54mm_Vertical -> Connector_PinHeader_2.54mm:PinHeader_1x03_P2.54mm_Vertical
Connections:
- net LCD_DC: now also J3.1 (Pin_1); no longer J3.3 (Pin_3)
- net LCD_RESET: now also J3.3 (Pin_3); no longer J3.1 (Pin_1)
Changed lines of the file:
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@@
 	)
 	(label "LCD_DC"
-		(at 35.56 36.83 0)
+		(at 35.56 31.75 0)
 		(effects
 			(font
@@
 	)
 	(label "LCD_RESET"
-		(at 35.56 31.75 0)
+		(at 35.56 36.83 0)
 		(effects
 			(font
@@
 			)
 		)
-		(property "Footprint" "Connector_PinHeader_2.54mm:PinHeader_1x02_P2.54mm_Vertical"
+		(property "Footprint" "Connector_PinHeader_2.54mm:PinHeader_1x03_P2.54mm_Vertical"
 			(at 60.96 34.29 0)
 			(effects
