File: Hardware_v2/oscar_components.kicad_pcb (KiCad board)
At the start: 4 copper layers, 71 x 100 mm, 64 parts, among them J1 SWD_Header, J10 USB_C_Receptacle, J2 ChannelA_In, J3 ChannelB_In, J4 ChannelC_In, J5 ChA_Buff_Out, J6 ChB_Buff_Out, J7 ChC_Buff_Out, J8 MIDI_IN, J9 Eurorack_10_pin_power, SW1 Left_Encoder, SW2 Right_Encoder, SW3 Reset_Button, U1 STM32F446RETx, U2 ILI9341_SPI_Daughterboard, U3 MCP6004, U4 TL074, U5 LT1117-3.3, U6 6N137, Y1 8MHz

Commit message: Routing of component board
Parts:
- added SW4: Menu_Button, Button_Switch_THT:SW_PUSH_6mm, F.Cu at (132.2, 106.0)
- C11: value 10uF -> 4.7uF; footprint Capacitor_SMD:CP_Elec_4x5.8 -> Capacitor_SMD:C_0805_2012Metric
- J11: renamed from J8; value MIDI_IN -> MIDI_OUT
- SW3: footprint Buttons_Switches_THT:SW_PUSH_6mm -> Button_Switch_THT:SW_PUSH_6mm
- U2: footprint Custom_Footprints:ILI9341_SPI_daughterboard -> Custom_Footprints:ILI9341_SPI_daughterboard_v2
- Y1: footprint Crystal:Crystal_SMD_Abracon_ABM3-2Pin_5.0x3.2mm -> Custom_Footprints:Crystal_SMD_5032-2Pin_5.0x3.2mm_Large_Pads
- moved R20 46.5 mm to (145.7, 116.6)
- moved C11 39.5 mm to (114.9, 76.3), turned to 0 degrees
- moved R13 32.3 mm to (109.0, 56.9), turned to -90 degrees
- moved J1 30.5 mm to (166.2, 63.6), turned to -90 degrees
- moved C14 29.0 mm to (158.2, 57.3), turned to 90 degrees
- moved R15 25.6 mm to (136.6, 84.0), turned to 90 degrees
- moved C9 7.18 mm to (146.9, 84.0), turned to -90 degrees
- moved U5 6.70 mm to (151.1, 56.7)
- moved D4 4.76 mm to (145.7, 113.4), turned to 0 degrees
- moved U6 3.04 mm to (145.7, 99.6), turned to 90 degrees
- moved R14 1.71 mm to (145.7, 110.4), turned to 0 degrees
- moved R16 1.20 mm to (114.9, 78.4)
- moved R17 1.20 mm to (114.9, 80.4)
- moved C2 0.95 mm to (153.2, 87.8)
- moved C3 0.95 mm to (149.6, 87.8)
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Connections:
- C11 pad 1: +12V -> -12V
- D3 pad 1: /USB_D+ -> /USB_DM
- D3 pad 2: /USB_D- -> /USB_DP
- J10 pad A6: /USB_D+ -> /USB_DP
- J10 pad A7: /USB_D- -> /USB_DM
- J10 pad B6: /USB_D+ -> /USB_DP
- J10 pad B7: /USB_D- -> /USB_DM
- J11 pad S: unconnected-(J8-PadS) -> unconnected-(J11-PadS)
- J2 pad 3: /CHB_In -> /CHA_In
- J3 pad 3: /CHC_In -> /CHB_In
- J4 pad 3: /CHA_In -> /CHC_In
- R2 pad 2: /CHA_In -> /CHC_In
- R4 pad 2: /CHB_In -> /CHA_In
- R6 pad 2: /CHC_In -> /CHB_In
- U1 pad 15: unconnected-(U1-PA1-Pad15) -> /MIDI_RX
- U1 pad 16: unconnected-(U1-PA2-Pad16) -> /MENU
- U1 pad 17: unconnected-(U1-PA3-Pad17) -> /ChC_Button
- U1 pad 2: /LCD_DC -> /R_ENC_BTN
- U1 pad 26: unconnected-(U1-PB0-Pad26) -> /ChB_Button
- U1 pad 27: unconnected-(U1-PB1-Pad27) -> /L_ENC_BTN
- U1 pad 3: /LCD_RESET -> unconnected-(U1-PC14-Pad3)
- U1 pad 33: unconnected-(U1-PB12-Pad33) -> /ChB_LED
- U1 pad 34: /R_ENC_BTN -> /ChA_LED
- U1 pad 35: unconnected-(U1-PB14-Pad35) -> /ChA_Button
- U1 pad 36: unconnected-(U1-PB15-Pad36) -> /ChC_LED
- U1 pad 37: /R_ENC_UP -> unconnected-(U1-PC6-Pad37)
- U1 pad 38: /R_ENC_DN -> unconnected-(U1-PC7-Pad38)
- U1 pad 41: unconnected-(U1-PA8-Pad41) -> /LCD_DC
- U1 pad 43: /L_ENC_BTN -> /LCD_RESET
- U1 pad 52: /MIDI_RX -> unconnected-(U1-PC11-Pad52)
- U1 pad 58: /L_ENC_UP -> /R_ENC_UP
- U1 pad 59: /L_ENC_DN -> /R_ENC_DN
- U1 pad 61: unconnected-(U1-PB8-Pad61) -> /L_ENC_UP
- U1 pad 62: unconnected-(U1-PB9-Pad62) -> /L_ENC_DN
- U2 pad 1: GND -> /LCD_DC
- U2 pad 10: GND -> +3.3V
- U2 pad 2: /LCD_RESET -> GND
- U2 pad 3: /LCD_SCK -> /LCD_RESET
- U2 pad 4: /LCD_DC -> /LCD_SCK
- U2 pad 5: /LCD_MOSI -> GND
- U2 pad 6: GND -> /LCD_MOSI
- U2 pad 7: Net-(U2-BackLight) -> GND
- U2 pad 8: GND -> Net-(U2-BackLight)
- U2 pad 9: +3.3V -> GND
- U4 pad 10: /CHA_In -> /CHC_In
- U4 pad 3: /CHC_In -> /CHB_In
- U4 pad 5: /CHB_In -> /CHA_In
Routing:
- net +3.3V: track 15.0 -> 202.1 mm, vias 0 -> 28
- net /USB_DP: track 0.00 -> 133.4 mm, vias 0 -> 1
- net /USB_DM: track 0.00 -> 126.6 mm, vias 0 -> 1
- net /ChA_Button: track 0.00 -> 107.2 mm
- net /ChB_Button: track 0.00 -> 107.1 mm
- net +12V: track 0.00 -> 95.7 mm, vias 0 -> 2
- net /L_ENC_UP: track 0.00 -> 94.3 mm, vias 0 -> 1
- net /L_ENC_DN: track 0.00 -> 84.6 mm, vias 0 -> 1
- net /ChC_LED: track 0.00 -> 76.8 mm, vias 0 -> 2
- net /L_ENC_BTN: track 0.00 -> 73.1 mm
- net /ChB_LED: track 0.00 -> 66.5 mm
- net /ChA_LED: track 0.00 -> 65.9 mm
- net +3.3VA: track 9.75 -> 74.2 mm, vias 1 -> 3
- net /NRST: track 0.00 -> 62.4 mm, vias 0 -> 1
- net /R_ENC_DN: track 0.00 -> 59.7 mm
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- added copper zone on B.Cu, net +3.3V
- added copper zone on F.Cu, net +3.3V
- added copper zone on In1.Cu, net +3.3V
- added copper zone on In2.Cu, net +3.3V
- added copper zone on B.Cu, net GND
- added copper zone on F.Cu, net GND
- added copper zone on In1.Cu, net GND
- added copper zone on In2.Cu, net GND
- removed copper zone on B.Cu, net +3.3VA
- removed copper zone on F.Cu, net +3.3VA
- removed copper zone on In1.Cu, net +3.3VA
- removed copper zone on In2.Cu, net +3.3VA
Other:
- board text removed: "-12V"
- board text removed: "12V"
- board text removed: "3.3V"
- board text removed: "CLK"
- board text removed: "Channel A"
- board text removed: "Channel B"
- board text removed: "Channel C"
- board text removed: "DC"
- board text removed: "GND"
- board text removed: "IO"
- board text removed: "MIDI"
- board text removed: "MOSI"
- board text removed: "RS"
- board text removed: "Reset"
- board text removed: "SCK"
