File: Hardware_v2/oscar_components.kicad_sch (KiCad schematic)
At the start: 64 parts, among them J1 SWD_Header, J10 USB_C_Receptacle, J2 ChannelA_In, J3 ChannelB_In, J4 ChannelC_In, J5 ChA_Buff_Out, J6 ChB_Buff_Out, J7 ChC_Buff_Out, J8 MIDI_IN, J9 Eurorack_10_pin_power, SW1 Left_Encoder, SW2 Right_Encoder, SW3 Reset_Button, SW4 Menu_Button, U1 STM32F446RETx, U2 ILI9341_SPI_Daughterboard, U3 MCP6004, U4 TL074, U5 LT1117-3.3, U6 6N137, Y1 8MHz

Commit message: Routing of component board
Parts:
- added J11: MIDI_OUT, Custom_Footprints:Thonkiconn_Stereo-PJ366ST, symbol thonkiconn:AudioJack3
- C11: value 10uF -> 4.7uF; footprint Capacitor_SMD:CP_Elec_4x5.8 -> Capacitor_SMD:C_0805_2012Metric
- SW3, SW4: footprint Buttons_Switches_THT:SW_PUSH_6mm -> Button_Switch_THT:SW_PUSH_6mm
- U2: footprint Custom_Footprints:ILI9341_SPI_daughterboard -> Custom_Footprints:ILI9341_SPI_daughterboard_v2
Connections:
- net +12V: no longer C11.1
- net +3.3V: now also U2.10 (3V3); no longer U2.9 (3V3)
- net -12V: now also C11.1
- net CHA_In: now also J2.3, R4.2, U4.5 (+); no longer J4.3, R2.2, U4.10 (+)
- net CHB_In: now also J3.3, R6.2, U4.3 (+); no longer J2.3, R4.2, U4.5 (+)
- net CHC_In: now also J4.3, R2.2, U4.10 (+); no longer J3.3, R6.2, U4.3 (+)
- net ChA_Button: now also U1.35 (PB14)
- net ChA_LED: now also U1.34 (PB13)
- net ChB_Button: now also U1.26 (PB0)
- net ChB_LED: now also U1.33 (PB12)
- net ChC_Button: now also U1.17 (PA3)
- net ChC_LED: now also U1.36 (PB15)
- net GND: now also U2.2 (GND), U2.5 (GND), U2.7 (GND), U2.9 (GND); no longer U2.1 (GND), U2.10 (GND), U2.6 (GND), U2.8 (GND)
- net LCD_DC: now also U1.41 (PA8), U2.1 (DC); no longer U1.2 (PC13), U2.4 (DC)
- net LCD_MOSI: now also U2.6 (MOSI); no longer U2.5 (MOSI)
- net LCD_RESET: now also U1.43 (PA10), U2.3 (RESET); no longer U1.3 (PC14), U2.2 (RESET)
- net LCD_SCK: now also U2.4 (SCK); no longer U2.3 (SCK)
- net L_ENC_BTN: now also U1.27 (PB1); no longer U1.43 (PA10)
- net L_ENC_DN: now also U1.62 (PB9); no longer U1.59 (PB7)
- net L_ENC_UP: now also U1.61 (PB8); no longer U1.58 (PB6)
- net MIDI_DATA: now also J11.T
- net MIDI_RX: now also U1.15 (PA1); no longer U1.52 (PC11)
- net MIDI_VREF: now also J11.R
- net NRST: no longer SW4.1
- net R_ENC_BTN: now also U1.2 (PC13); no longer U1.34 (PB13)
- net R_ENC_DN: now also U1.59 (PB7); no longer U1.38 (PC7)
- net R_ENC_UP: now also U1.58 (PB6); no longer U1.37 (PC6)
- net USB_DM: now also D3.1 (K1), J10.A7 (D-), J10.B7 (D-)
- net USB_DP: now also D3.2 (K2), J10.A6 (D+), J10.B6 (D+)
- net MENU: now reaches U1.16 (PA2)
- net MENU: now also SW4.1
- net at R13.2: now also U2.8 (BackLight); no longer U2.7 (BackLight)
- removed net USB_D+: D3.1 (K1), J10.A6 (D+), J10.B6 (D+)
- removed net USB_D-: D3.2 (K2), J10.A7 (D-), J10.B7 (D-)
- no-connect marks 50 -> 43
Other:
- moved on the sheet: C12, R13
